Commit message: Add stable UGV01-X3 web mapping dashboard baseline

File: urdf/ugv01_box.urdf (robot description, URDF)
Before this commit: robot ugv01_box_light, 3 links, 2 joints
Links:
- removed link ldlidar_link
- added link antenna_base; visual cylinder length=0.018 radius=0.009
- added link antenna_whip; visual cylinder length=0.165 radius=0.003
- added link front_camera_lens; visual cylinder length=0.010 radius=0.013
- added link front_left_light; visual cylinder length=0.008 radius=0.010
- added link front_right_light; visual cylinder length=0.008 radius=0.010
- added link front_sensor_bar; visual box size=0.024 0.088 0.026
- added link ldlidar_base; visual cylinder length=0.006 radius=0.019; visual cylinder length=0.018 radius=0.025
- added link left_front_sprocket; visual cylinder length=0.040 radius=0.021
- added link left_rear_sprocket; visual cylinder length=0.040 radius=0.021
- added link left_road_wheels; visual cylinder length=0.036 radius=0.014; visual cylinder length=0.036 radius=0.014
- added link left_side_armor; visual box size=0.178 0.008 0.066
- added link left_side_slot_1; visual box size=0.050 0.004 0.006
- added link left_track_lower; visual box size=0.218 0.040 0.018
- added link left_track_upper; visual box size=0.196 0.038 0.020
- added link left_tread_blocks; visual box size=0.012 0.046 0.010; visual box size=0.012 0.046 0.010
- added link right_front_sprocket; visual cylinder length=0.040 radius=0.021
- added link right_rear_sprocket; visual cylinder length=0.040 radius=0.021
- added link right_road_wheels; visual cylinder length=0.036 radius=0.014; visual cylinder length=0.036 radius=0.014
- added link right_side_armor; visual box size=0.178 0.008 0.066
- added link right_side_slot_1; visual box size=0.050 0.004 0.006
- added link right_track_lower; visual box size=0.218 0.040 0.018
- added link right_track_upper; visual box size=0.196 0.038 0.020
- added link right_tread_blocks; visual box size=0.012 0.046 0.010; visual box size=0.012 0.046 0.010
- added link status_led; visual sphere radius=0.006
- added link top_plate; visual box size=0.162 0.116 0.012
- added link top_rail_front; visual box size=0.170 0.008 0.012
- added link top_rail_rear; visual box size=0.170 0.008 0.012
- link base_link: geometry collision box size=0.232 0.197 0.110; visual box size=0.168 0.120 0.010
Joints:
- removed joint base_link_to_ldlidar_link
- added joint antenna_base_joint: type fixed, parent base_link, child antenna_base, origin xyz=-0.088 0.058 0.126 rpy=0 0 0
- added joint antenna_whip_joint: type fixed, parent antenna_base, child antenna_whip, origin xyz=0 0 0.010 rpy=0 0 0
- added joint base_link_to_ldlidar_base: type fixed, parent base_link, child ldlidar_base, origin xyz=0.045 0.000 0.123 rpy=0 0 1.5708
- added joint base_to_left_side_armor: type fixed, parent base_link, child left_side_armor, origin xyz=0.000 0.071 0.060 rpy=0 0 0
- added joint base_to_left_track_lower: type fixed, parent base_link, child left_track_lower, origin xyz=0.000 0.098 0.015 rpy=0 0 0
- added joint base_to_left_track_upper: type fixed, parent base_link, child left_track_upper, origin xyz=0.000 0.098 0.064 rpy=0 0 0
- added joint base_to_right_side_armor: type fixed, parent base_link, child right_side_armor, origin xyz=0.000 -0.071 0.060 rpy=0 0 0
- added joint base_to_right_track_lower: type fixed, parent base_link, child right_track_lower, origin xyz=0.000 -0.098 0.015 rpy=0 0 0
- added joint base_to_right_track_upper: type fixed, parent base_link, child right_track_upper, origin xyz=0.000 -0.098 0.064 rpy=0 0 0
- added joint base_to_top_plate: type fixed, parent base_link, child top_plate, origin xyz=0.015 0 0.118 rpy=0 0 0
- added joint front_camera_lens_joint: type fixed, parent base_link, child front_camera_lens, origin xyz=0.131 0.000 0.075 rpy=0 0 0
- added joint front_left_light_joint: type fixed, parent base_link, child front_left_light, origin xyz=0.131 0.032 0.077 rpy=0 0 0
- added joint front_right_light_joint: type fixed, parent base_link, child front_right_light, origin xyz=0.131 -0.032 0.077 rpy=0 0 0
- added joint front_sensor_bar_joint: type fixed, parent base_link, child front_sensor_bar, origin xyz=0.117 0 0.075 rpy=0 0 0
- added joint left_front_sprocket_joint: type fixed, parent base_link, child left_front_sprocket, origin xyz=0.095 0.098 0.034 rpy=0 0 0
- added joint left_rear_sprocket_joint: type fixed, parent base_link, child left_rear_sprocket, origin xyz=-0.095 0.098 0.034 rpy=0 0 0
- added joint left_road_wheels_joint: type fixed, parent base_link, child left_road_wheels, origin xyz=0.000 0.098 0.030 rpy=0 0 0
- added joint left_side_slot_1_joint: type fixed, parent base_link, child left_side_slot_1, origin xyz=-0.030 0.076 0.060 rpy=0 0 0
- added joint left_tread_blocks_joint: type fixed, parent base_link, child left_tread_blocks, origin xyz=0.000 0.098 0.006 rpy=0 0 0
- added joint right_front_sprocket_joint: type fixed, parent base_link, child right_front_sprocket, origin xyz=0.095 -0.098 0.034 rpy=0 0 0
- added joint right_rear_sprocket_joint: type fixed, parent base_link, child right_rear_sprocket, origin xyz=-0.095 -0.098 0.034 rpy=0 0 0
- added joint right_road_wheels_joint: type fixed, parent base_link, child right_road_wheels, origin xyz=0.000 -0.098 0.030 rpy=0 0 0
- added joint right_side_slot_1_joint: type fixed, parent base_link, child right_side_slot_1, origin xyz=-0.030 -0.076 0.060 rpy=0 0 0
- added joint right_tread_blocks_joint: type fixed, parent base_link, child right_tread_blocks, origin xyz=0.000 -0.098 0.006 rpy=0 0 0
- added joint status_led_joint: type fixed, parent base_link, child status_led, origin xyz=0.048 0.000 0.156 rpy=0 0 0
- added joint top_rail_front_joint: type fixed, parent base_link, child top_rail_front, origin xyz=0.012 0.064 0.123 rpy=0 0 0
- added joint top_rail_rear_joint: type fixed, parent base_link, child top_rail_rear, origin xyz=0.012 -0.064 0.123 rpy=0 0 0
- joint base_footprint_to_base_link: origin xyz=0 0 0 rpy=0 0 -1.5708 -> xyz=0 0 0 rpy=0 0 0
